File: PCB/Daughterboard/Daughterboard.sch (EAGLE design)
At the start: 12 parts, among them U3 VCNL4020-GS08, U5 NC7SZ08M5X

Commit message: PCB rev2 uploaded
Other:
- note added: "REV 1"
Changed lines of the file:
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@@
 <part name="R28" library="rcl" deviceset="R-EU_" device="R0603" value="100k"/>
 <part name="JP2" library="pinhead" deviceset="PINHD-1X20" device="/90"/>
+<part name="FRAME1" library="frames" deviceset="A4L-LOC" device=""/>
+<part name="FRAME2" library="frames" deviceset="A4L-LOC" device=""/>
 </parts>
 <sheets>
@@
 <text x="53.34" y="0" size="1.27" layer="91" rot="R90">Sensor Expansion Port (out)</text>
 <text x="-5.08" y="0" size="1.27" layer="91" rot="R90">Sensor Expansion Port (in)</text>
+<text x="146.304" y="-96.266" size="1.778" layer="94">REV 1</text>
 </plain>
 <instances>
@@
 <instance part="R28" gate="G$1" x="-38.1" y="-30.48" rot="R90"/>
 <instance part="JP2" gate="A" x="0" y="10.16" rot="MR0"/>
+<instance part="FRAME1" gate="G$1" x="-101.6" y="-101.6"/>
+<instance part="FRAME2" gate="G$1" x="-101.6" y="-101.6"/>
 </instances>
 <busses>
