File: PCB/Mainboard/Doorbell.brd (EAGLE design)
At the start: 95.7 x 77.4 mm, 99 parts, among them IC1 CP2104-F03-GM, J1 105017-1001, J2 FH12A-24S-0.5SH(55), Q1 PMF370XN, U1 ESP-WROOM-32, U2 TCA9548APWR, U3 VCNL4020-GS08, U4 MCP73831T-2ACI/OT, U5 NC7SZ08M5X, U6 TPS61200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

Commit message: PCB rev2 uploaded
Parts:
- C16: value 4.7uF -> 1uF
- C18: value 10u -> 10uF
- C21: value 100n -> 100nF
- R16: value 1.2M -> 1M
- R17: value 220k -> 180k
- R20: value 220k -> 150k
- R21: value 2M -> 1M
- R25, R26: value 0R -> DO NOT FIT - 0R
- R27: value 10k -> DO NOT FIT - 10k
- R31, R32, R33, R34: value 10k -> 2k7
- U7: value AP2112-3.3 -> AP2112-3.3 - DO NOT FIT
Changed lines of the file:
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@@
 <attribute name="NAME" x="69.862209375" y="52.541340625" size="0.8128" layer="26" rot="MR0"/>
 </element>
-<element name="C16" library="rcl" package="C0603" value="4.7uF" x="62.090409375" y="46.780215625" smashed="yes" rot="MR0">
+<element name="C16" library="rcl" package="C0603" value="1uF" x="62.090409375" y="46.780215625" smashed="yes" rot="MR0">
 <attribute name="NAME" x="62.979409375" y="47.669215625" size="0.8128" layer="26" rot="MR0"/>
 </element>
@@
 <attribute name="NAME" x="18.234471875" y="61.65724375" size="0.8128" layer="26" rot="MR180"/>
 </element>
-<element name="C18" library="rcl" package="C1206" value="10u" x="27.94" y="62.23" smashed="yes" rot="MR90">
+<element name="C18" library="rcl" package="C1206" value="10uF" x="27.94" y="62.23" smashed="yes" rot="MR90">
 <attribute name="NAME" x="29.21" y="62.357" size="0.8128" layer="26" rot="MR90"/>
 </element>
@@
 <attribute name="NAME" x="48.558596875" y="58.695303125" size="0.8128" layer="26" rot="MR90"/>
 </element>
-<element name="R16" library="rcl" package="R0603" value="1.2M" x="50.95875" y="66.04" smashed="yes" rot="MR90">
+<element name="R16" library="rcl" package="R0603" value="1M" x="50.95875" y="66.04" smashed="yes" rot="MR90">
 <attribute name="NAME" x="50.495715625" y="67.73520625" size="0.8128" layer="26" rot="MR90"/>
 </element>
-<element name="R17" library="rcl" package="R0603" value="220k" x="48.895" y="66.04" smashed="yes" rot="MR270">
+<element name="R17" library="rcl" package="R0603" value="180k" x="48.895" y="66.04" smashed="yes" rot="MR270">
 <attribute name="NAME" x="49.3279" y="69.995803125" size="0.8128" layer="26" rot="MR270"/>
 </element>
@@
 <attribute name="NAME" x="50.83780625" y="59.858790625" size="0.8128" layer="26" rot="MR180"/>
 </element>
-<element name="R20" library="rcl" package="R0603" value="220k" x="45.72" y="67.31" smashed="yes" rot="MR180">
+<element name="R20" library="rcl" package="R0603" value="150k" x="45.72" y="67.31" smashed="yes" rot="MR180">
 <attribute name="NAME" x="44.60875" y="69.215" size="0.8128" layer="26" rot="MR180"/>
 </element>
-<element name="R21" library="rcl" package="R0603" value="2M" x="41.91" y="67.31" smashed="yes" rot="MR0">
+<element name="R21" library="rcl" package="R0603" value="1M" x="41.91" y="67.31" smashed="yes" rot="MR0">
 <attribute name="NAME" x="40.3225" y="66.9925" size="0.8128" layer="26" rot="MR0"/>
 </element>
-<element name="C21" library="rcl" package="C0603" value="100n" x="42.545" y="62.38875" smashed="yes" rot="MR90">
+<element name="C21" library="rcl" package="C0603" value="100nF" x="42.545" y="62.38875" smashed="yes" rot="MR90">
 <attribute name="NAME" x="41.5925" y="62.70625" size="0.8128" layer="26" rot="MR0"/>
 </element>
@@
 <attribute name="NAME" x="42.9278" y="56.62" size="0.8128" layer="26" rot="MR180"/>
 </element>
-<element name="U7" library="microbuilder" package="SOT23-5" value="AP2112-3.3" x="44.45" y="53.975" smashed="yes" rot="MR90">
+<element name="U7" library="microbuilder" package="SOT23-5" value="AP2112-3.3 - DO NOT FIT" x="44.45" y="53.975" smashed="yes" rot="MR90">
 <attribute name="NAME" x="43.942" y="53.159" size="0.8128" layer="26" ratio="18" rot="MR90"/>
 </element>
-<element name="R25" library="rcl" package="R0603" value="0R" x="38.1" y="53.975" smashed="yes" rot="MR90">
+<element name="R25" library="rcl" package="R0603" value="DO NOT FIT - 0R" x="38.1" y="53.975" smashed="yes" rot="MR90">
 <attribute name="NAME" x="36.449" y="52.832" size="0.8128" layer="26" rot="MR90"/>
 </element>
-<element name="R26" library="rcl" package="R0603" value="0R" x="48.26" y="53.975" smashed="yes" rot="MR90">
+<element name="R26" library="rcl" package="R0603" value="DO NOT FIT - 0R" x="48.26" y="53.975" smashed="yes" rot="MR90">
 <attribute name="NAME" x="46.609" y="52.832" size="0.8128" layer="26" rot="MR90"/>
 </element>
-<element name="R27" library="rcl" package="R0603" value="10k" x="40.64" y="53.975" smashed="yes" rot="MR270">
+<element name="R27" library="rcl" package="R0603" value="DO NOT FIT - 10k" x="40.64" y="53.975" smashed="yes" rot="MR270">
 <attribute name="NAME" x="42.291" y="55.118" size="0.8128" layer="26" rot="MR270"/>
 </element>
@@
 <attribute name="VALUE" x="73.93" y="24.67" size="1.27" layer="27"/>
 </element>
-<element name="R31" library="rcl" package="R0603" value="10k" x="48.26" y="29.21" smashed="yes" rot="R180">
+<element name="R31" library="rcl" package="R0603" value="2k7" x="48.26" y="29.21" smashed="yes" rot="R180">
 <attribute name="NAME" x="49.277959375" y="31.330640625" size="0.8128" layer="25" rot="R180"/>
 </element>
-<element name="R32" library="rcl" package="R0603" value="10k" x="57.15" y="29.21" smashed="yes" rot="R180">
+<element name="R32" library="rcl" package="R0603" value="2k7" x="57.15" y="29.21" smashed="yes" rot="R180">
 <attribute name="NAME" x="58.313846875" y="31.294175" size="0.8128" layer="25" rot="R180"/>
 </element>
-<element name="R33" library="rcl" package="R0603" value="10k" x="66.04" y="29.21" smashed="yes" rot="R180">
+<element name="R33" library="rcl" package="R0603" value="2k7" x="66.04" y="29.21" smashed="yes" rot="R180">
 <attribute name="NAME" x="67.076196875" y="31.312409375" size="0.8128" layer="25" rot="R180"/>
 </element>
-<element name="R34" library="rcl" package="R0603" value="10k" x="74.93" y="29.21" smashed="yes" rot="R180">
+<element name="R34" library="rcl" package="R0603" value="2k7" x="74.93" y="29.21" smashed="yes" rot="R180">
 <attribute name="NAME" x="76.0756125" y="31.312409375" size="0.8128" layer="25" rot="R180"/>
 </element>
